File: pcb/misa.kicad_sch (KiCad schematic)
At the start: 2 parts, among them U1 MC68000P

Commit message: mega stuff
Parts:
- added C2, C4, C5, C6, C7: 100n, symbol Device:C
- added C3: 1u, symbol Device:C_Polarized
- added R1, R2: 1M, symbol Device:R
- added R10, R11, R12, R3, R4, R5, R6, R7, R8, R9: 10K, symbol Device:R
- added SW1: Reset, symbol Switch:SW_Push
- added U2: NE555P, Package_DIP:DIP-8_W7.62mm, symbol Timer:NE555P
- added U3: 74LS148, symbol 74xx:74LS148
- added U4: 74HC74, symbol 74xx:74HC74
- added U5: 74LS05, symbol 74xx:74LS05
- added U6: 74LS10, symbol 74xx:74LS10
- added Y1: 8MHz, Oscillator:Oscillator_DIP-8, symbol Oscillator:CXO_DIP8
Connections:
- net +5V: now also C4.1, C5.1, C6.1, C7.1, R1.1, R10.1, R11.1, R12.1, R2.2, R3.1, R4.1, R5.1, R6.1, R7.1, R8.1, R9.1, U2.4 (R), U2.8 (VCC), U3.16 (VCC), U4.1 (~{R}), U4.10 (~{S}), U4.13 (~{R}), U4.14 (VCC), U4.4 (~{S}), U5.14 (VCC), U6.14 (VCC), Y1.8 (Vcc)
- net GND: now also C2.2, C3.2, C4.2, C5.2, C6.2, C7.2, SW1.1, U2.1 (GND), U2.5 (CV), U3.10 (IO), U3.5 (EI), U3.8 (GND), U4.7 (GND), U5.7 (GND), U6.7 (GND), Y1.4 (GND)
- net HALT: now reaches U1.17 (~{HALT})
- net HALT: now also R4.2, U5.4
- net RESET: now reaches U1.18 (~{RESET})
- net RESET: now also R3.2, U5.2
- new net: C3.1, R2.1, U2.6 (THR), U2.7 (DIS)
- new net: C2.1, R1.2, SW1.2, U2.2 (TR)
- new net: U2.3 (Q), U5.1, U5.3
- new net: U4.12 (D), U4.8 (~{Q})
- new net: U4.2 (D), U4.6 (~{Q})
- new net: R5.2, Y1.1 (EN)
- new net 1/2CLOCK: U4.11 (C), U4.5 (Q)
- new net 1/4CLOCK: U4.9 (Q)
- new net CLOCK: U4.3 (C), Y1.5 (OUT)
- new net FC0: U6.1
- new net FC1: U6.2
- new net FC2: U6.13
- new net IPL0: U3.9 (S0)
- new net IPL1: U3.7 (S1)
- new net IPL2: U3.6 (S2)
- new net IRQ1: R10.2, R11.2, R12.2, R6.2, R7.2, R8.2, R9.2, U3.1 (I4), U3.11 (I1), U3.12 (I2), U3.13 (I3), U3.2 (I5), U3.3 (I6), U3.4 (I7)
- new net VPA: U6.12
Other:
- note added: "CLOCK"
- note added: "INTERRUPT"
- note added: "RESET"

Commit message: mega stuff
Parts:
- added C10, C11, C12, C13, C8, C9: 100n, symbol Device:C
- added D1: RUN, symbol Device:LED
- added J1: 1/1CLOCK, symbol Connector:Conn_01x02_Pin
- added J2: 1/2CLOCK, symbol Connector:Conn_01x02_Pin
- added J3: 1/4CLOCK, symbol Connector:Conn_01x02_Pin
- added R13: 220R, symbol Device:R
- added U10, U7, U8, U9: AS6C4008-55PCN, Package_DIP:DIP-32_W15.24mm, symbol Memory_RAM:AS6C4008-55PCN
- added U11, U12: SST39SF040, symbol Memory_Flash:SST39SF040
Connections:
- net +5V: now also C10.1, C11.1, C12.1, C13.1, C8.1, C9.1, D1.2 (A), U10.32 (VCC), U11.32 (VCC), U12.32 (VCC), U7.32 (VCC), U8.32 (VCC), U9.32 (VCC)
- net 1/2CLOCK: now also J2.1 (Pin_1)
- net 1/4CLOCK: now also J3.1 (Pin_1)
- net FC0: now also U1.28 (FC0)
- net FC1: now also U1.27 (FC1)
- net FC2: now also U1.26 (FC2)
- net GND: now also C10.2, C11.2, C12.2, C13.2, C8.2, C9.2, U10.16 (VSS), U11.16 (GND), U12.16 (GND), U7.16 (VSS), U8.16 (VSS), U9.16 (VSS)
- net HALT: now also U5.5
- net IPL0: now also U1.25 (~{IPL0})
- net IPL1: now also U1.24 (~{IPL1})
- net IPL2: now also U1.23 (~{IPL2})
- net IRQ1: no longer R10.2, R11.2, R12.2, R7.2, R8.2, R9.2, U3.1 (I4), U3.12 (I2), U3.13 (I3), U3.2 (I5), U3.3 (I6), U3.4 (I7)
- net VPA: now also U1.21 (~{VPA})
- net MPUCLOCK: now reaches U1.15 (CLK)
- net MPUCLOCK: now also J1.2 (Pin_2), J2.2 (Pin_2), J3.2 (Pin_2)
- net CLOCK renamed 1/1CLOCK
- net 1/1CLOCK: now also J1.1 (Pin_1)
- new net: D1.1 (K), R13.2
- new net: R13.1, U5.6
- new net IRQ2: R7.2, U3.12 (I2)
- new net IRQ3: R8.2, U3.13 (I3)
- new net IRQ4: R9.2, U3.1 (I4)
- new net IRQ5: R10.2, U3.2 (I5)
- new net IRQ6: R11.2, U3.3 (I6)
- new net IRQ7: R12.2, U3.4 (I7)
Other:
- moved on the sheet: C2, C3, C7, R1, R10, R11, R12, R2, R3, R4, R5, R6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

Commit message: mega stuff
Parts:
- removed J1: 1/1CLOCK, symbol Connector:Conn_01x02_Pin
- removed J2: 1/2CLOCK, symbol Connector:Conn_01x02_Pin
- removed J3: 1/4CLOCK, symbol Connector:Conn_01x02_Pin
- added C14, C15, C16, C17, C18, C19, C20, C21: 100n, symbol Device:C
- added JP2, JP3, JP4: Jumper_2_Open, symbol Jumper:Jumper_2_Open
- added R14: 10K, symbol Device:R
- added U13, U14: SST39SF040, symbol Memory_Flash:SST39SF040
- added U15: 74HCT138, symbol 74xx:74HCT138
- added U16: 74LS175, symbol 74xx:74LS175
- added U17: 74LS390, symbol 74xx:74LS390
- added U18, U20: 74LS08, symbol 74xx:74LS08
- added U19: 74HCT04, symbol 74xx:74HCT04
Connections:
- net +5V: now also C14.1, C15.1, C16.1, C17.1, C18.1, C19.1, C20.1, C21.1, R14.1, U13.32 (VCC), U14.32 (VCC), U15.16 (VCC), U16.16 (VCC), U17.16 (VCC), U18.14 (VCC), U19.14 (VCC), U20.14 (VCC)
- net 1/1CLOCK: now also JP2.1 (A)
- net 1/2CLOCK: now also JP3.1 (A)
- net 1/4CLOCK: now also JP4.1 (A)
- net GND: now also C14.2, C15.2, C16.2, C17.2, C18.2, C19.2, C20.2, C21.2, U13.16 (GND), U14.16 (GND), U15.5 (~{E1}), U15.6 (E2), U15.8 (GND), U16.8 (GND), U17.14 (MR), U17.2 (MR), U17.8 (GND), U18.7 (GND), U19.7 (GND), U20.7 (GND)
- net MPUCLOCK: now also JP2.2 (B), JP3.2 (B), JP4.2 (B), U17.1 (~{CP0})
- net D0: now reaches U7.13 (DQ0)
- net D0: now also U1.5 (D0), U11.13 (D0), U9.13 (DQ0), U13.13 (D0)
- net D1: now reaches U7.14 (DQ1)
- net D1: now also U1.4 (D1), U11.14 (D1), U9.14 (DQ1), U13.14 (D1)
- net D2: now reaches U7.15 (DQ2)
- net D2: now also U1.3 (D2), U11.15 (D2), U9.15 (DQ2), U13.15 (D2)
- net D3: now reaches U7.17 (DQ3)
- net D3: now also U1.2 (D3), U11.17 (D3), U9.17 (DQ3), U13.17 (D3)
- net D4: now reaches U7.18 (DQ4)
- net D4: now also U1.1 (D4), U11.18 (D4), U9.18 (DQ4), U13.18 (D4)
- net D5: now reaches U7.19 (DQ5)
- net D5: now also U1.64 (D5), U11.19 (D5), U9.19 (DQ5), U13.19 (D5)
- net D6: now reaches U7.20 (DQ6)
- net D6: now also U1.63 (D6), U11.20 (D6), U9.20 (DQ6), U13.20 (D6)
- net D7: now reaches U7.21 (DQ7)
- net D7: now also U1.62 (D7), U11.21 (D7), U9.21 (DQ7), U13.21 (D7)
- net RAM_CS: now reaches U7.22 (CE#)
- net RAM_CS: now also U10.22 (CE#), U8.22 (CE#), U9.22 (CE#), U15.14 (~{Y1})
- net D8: now reaches U8.13 (DQ0)
- net D8: now also U1.61 (D8), U10.13 (DQ0), U12.13 (D0), U14.13 (D0)
- net D9: now reaches U8.14 (DQ1)
- net D9: now also U1.60 (D9), U10.14 (DQ1), U12.14 (D1), U14.14 (D1)
- net D10: now reaches U8.15 (DQ2)
- net D10: now also U1.59 (D10), U10.15 (DQ2), U12.15 (D2), U14.15 (D2)
- net D11: now reaches U8.17 (DQ3)
- net D11: now also U1.58 (D11), U10.17 (DQ3), U12.17 (D3), U14.17 (D3)
- net D12: now reaches U8.18 (DQ4)
- net D12: now also U1.57 (D12), U10.18 (DQ4), U12.18 (D4), U14.18 (D4)
- net D13: now reaches U8.19 (DQ5)
- net D13: now also U1.56 (D13), U10.19 (DQ5), U12.19 (D5), U14.19 (D5)
- net D14: now reaches U8.20 (DQ6)
- net D14: now also U1.55 (D14), U10.20 (DQ6), U12.20 (D6), U14.20 (D6)
- net D15: now reaches U8.21 (DQ7)
- net D15: now also U1.54 (D15), U10.21 (DQ7), U12.21 (D7), U14.21 (D7)
- net BERR: now reaches U1.22 (~{BERR})
- net BERR: now also U16.14 (~{Q3})
- net A1: now reaches U1.29 (A1)
- net A2: now reaches U1.30 (A2)
- net A3: now reaches U1.31 (A3)
- net A4: now reaches U1.32 (A4)
- net A5: now reaches U1.33 (A5)
- net A6: now reaches U1.34 (A6)
- net A7: now reaches U1.35 (A7)
- net A8: now reaches U1.36 (A8)
- net A9: now reaches U1.37 (A9)
- net A10: now reaches U1.38 (A10)
- net A11: now reaches U1.39 (A11)
- net A12: now reaches U1.40 (A12)
- net A13: now reaches U1.41 (A13)
- net A14: now reaches U1.42 (A14)
- net A15: now reaches U1.43 (A15)
- net A16: now reaches U1.44 (A16)
- net A16: now also U19.11
- net A17: now reaches U1.45 (A17)
- net A17: now also U19.9
- net A18: now reaches U1.46 (A18)
- net A18: now also U19.5
- net A19: now reaches U1.47 (A19)
- net A19: now also U19.3
- net A20: now reaches U1.48 (A20)
- net A20: now also U15.1 (A0), U18.5
- net A21: now reaches U1.50 (A21)
- net A21: now also U15.2 (A1), U18.4
- net A22: now reaches U1.51 (A22)
- net A22: now also U15.3 (A2), U18.2
- net A23: now reaches U1.52 (A23)
- net A23: now also U18.1, U19.1
- net AS: now reaches U1.6 (~{AS})
- net AS: now also U5.9
- net UDS: now reaches U1.7 (~{UDS})
- net LDS: now reaches U1.8 (~{LDS})
- net ROM_CS: now reaches U12.22 (CE)
- net ROM_CS: now also U11.22 (CE), U13.22 (CE), U14.22 (CE), U15.15 (~{Y0})
- new net: U18.12, U19.4
- new net: U19.13, U20.8
- new net: U15.4 (~{E0}), U19.2
- new net: U19.8, U20.1
- new net: U18.10, U18.6
- new net: U18.11, U20.4
- new net: U20.3, U20.5
- new net: U20.10, U20.6
- new net: R14.2, U16.12 (D2), U5.8
- new net: U19.10, U20.2
- new net: U16.9 (Cp), U17.10 (Q2)
- new net: U18.13, U19.6
- new net: U17.3 (Q0), U17.4 (~{CP1})
- new net: U17.15 (~{CP0}), U17.7 (Q3)
- new net: U18.8, U20.9
- new net: U18.3, U18.9
- new net: U17.12 (~{CP1}), U17.13 (Q0)
- new net IO_CS: U19.12
Other:
- note added: "ADDRESS DECODER"
- note added: "BUS ERROR"
- note added: "MPU"
- note added: "RAM"
- note added: "ROM"
- moved on the sheet: C1, C10, C11, C12, C13, C2, C3, C4, C5, C6, C7, C8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

Commit message: mega stuff
Parts:
- removed C16, C17, C18, C19, C20, C21, C6, C7: 100n, symbol Device:C
- removed R10, R11, R12, R14, R6, R7, R8, R9: 10K, symbol Device:R
- removed U15: 74HCT138, symbol 74xx:74HCT138
- removed U16: 74LS175, symbol 74xx:74LS175
- removed U17: 74LS390, symbol 74xx:74LS390
- removed U18, U20: 74LS08, symbol 74xx:74LS08
- removed U19: 74HCT04, symbol 74xx:74HCT04
- removed U3: 74LS148, symbol 74xx:74LS148
- removed unit 1 of U5
- removed U6: 74LS10, symbol 74xx:74LS10
- added U21: ATF22V10, Package_DIP:DIP-24_W7.62mm_Socket, symbol my:ATF22V10
- added unit 3 of U5
Connections:
- net HALT: now also U5.5; no longer U5.5
- net RESET: now also U5.2
- net at U2.3 (Q), U5.3: now also U5.1
- net at R13.1: now also U5.6; no longer U5.6
- net ~{DTACK}: now reaches U1.10 (~{DTACK})
Other:
- note removed: "ADDRESS DECODER"
- note removed: "BUS ERROR"
- note removed: "INTERRUPT"
- moved on the sheet: C1, C10, C11, C12, C13, C14, C15, C2, C3, C5, C8, C9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

Commit message: mega stuff
Parts:
- added C6: 100n, symbol Device:C
Connections:
- net +5V: now also U21.24 (VCC), C6.1
- net GND: now also U21.12 (GND), C6.2
Other:
- note added: "PLD (ADDRESS DECODING, DTACK, BERR)"
- moved on the sheet: C4, C5, U21, U4C

Commit message: mega stuff
Connections:
- net AS is gone; now on net ~{AS}: U1.6 (~{AS})
- net BERR is gone; now on net ~{BERR}: U1.22 (~{BERR})
- net RAM_CS is gone; now on net ~{RAM_CS}: U10.22 (CE#), U7.22 (CE#), U8.22 (CE#), U9.22 (CE#)
- net ROM_CS is gone; now on net ~{ROM_CS}: U11.22 (CE), U12.22 (CE), U13.22 (CE), U14.22 (CE)
- net A1: now also U10.12 (A0), U11.12 (A0), U12.12 (A0), U13.12 (A0), U14.12 (A0), U7.12 (A0), U8.12 (A0), U9.12 (A0)
- net A10: now also U10.26 (A9), U11.26 (A9), U12.26 (A9), U13.26 (A9), U14.26 (A9), U7.26 (A9), U8.26 (A9), U9.26 (A9)
- net A11: now also U10.23 (A10), U11.23 (A10), U12.23 (A10), U13.23 (A10), U14.23 (A10), U7.23 (A10), U8.23 (A10), U9.23 (A10)
- net A12: now also U10.25 (A11), U11.25 (A11), U12.25 (A11), U13.25 (A11), U14.25 (A11), U7.25 (A11), U8.25 (A11), U9.25 (A11)
- net A13: now also U10.4 (A12), U11.4 (A12), U12.4 (A12), U13.4 (A12), U14.4 (A12), U7.4 (A12), U8.4 (A12), U9.4 (A12)
- net A14: now also U10.28 (A13), U11.28 (A13), U12.28 (A13), U13.28 (A13), U14.28 (A13), U7.28 (A13), U8.28 (A13), U9.28 (A13)
- net A15: now also U10.3 (A14), U11.29 (A14), U12.29 (A14), U13.29 (A14), U14.29 (A14), U7.3 (A14), U8.3 (A14), U9.3 (A14)
- net A16: now also U10.31 (A15), U11.3 (A15), U12.3 (A15), U13.3 (A15), U14.3 (A15), U21.9 (I), U7.31 (A15), U8.31 (A15), U9.31 (A15)
- net A17: now also U10.2 (A16), U11.2 (A16), U12.2 (A16), U13.2 (A16), U14.2 (A16), U21.8 (I), U7.2 (A16), U8.2 (A16), U9.2 (A16)
- net A18: now also U10.30 (A17), U11.30 (A17), U12.30 (A17), U13.30 (A17), U14.30 (A17), U21.7 (I), U7.30 (A17), U8.30 (A17), U9.30 (A17)
- net A19: now also U10.1 (A18), U11.1 (A18), U12.1 (A18), U13.1 (A18), U14.1 (A18), U21.6 (I), U7.1 (A18), U8.1 (A18), U9.1 (A18)
- net A2: now also U10.11 (A1), U11.11 (A1), U12.11 (A1), U13.11 (A1), U14.11 (A1), U7.11 (A1), U8.11 (A1), U9.11 (A1)
- net A20: now also U21.5 (I)
- net A21: now also U21.4 (I)
- net A22: now also U21.3 (I)
- net A23: now also U21.2 (I)
- net A3: now also U10.10 (A2), U11.10 (A2), U12.10 (A2), U13.10 (A2), U14.10 (A2), U7.10 (A2), U8.10 (A2), U9.10 (A2)
- net A4: now also U10.9 (A3), U11.9 (A3), U12.9 (A3), U13.9 (A3), U14.9 (A3), U7.9 (A3), U8.9 (A3), U9.9 (A3)
- net A5: now also U10.8 (A4), U11.8 (A4), U12.8 (A4), U13.8 (A4), U14.8 (A4), U7.8 (A4), U8.8 (A4), U9.8 (A4)
- net A6: now also U10.7 (A5), U11.7 (A5), U12.7 (A5), U13.7 (A5), U14.7 (A5), U7.7 (A5), U8.7 (A5), U9.7 (A5)
- net A7: now also U10.6 (A6), U11.6 (A6), U12.6 (A6), U13.6 (A6), U14.6 (A6), U7.6 (A6), U8.6 (A6), U9.6 (A6)
- net A8: now also U10.5 (A7), U11.5 (A7), U12.5 (A7), U13.5 (A7), U14.5 (A7), U7.5 (A7), U8.5 (A7), U9.5 (A7)
- net A9: now also U10.27 (A8), U11.27 (A8), U12.27 (A8), U13.27 (A8), U14.27 (A8), U7.27 (A8), U8.27 (A8), U9.27 (A8)
- net RESET: now also U2.3 (Q), U21.11 (I), U5.1, U5.3; no longer R3.2, U1.18 (~{RESET}), U5.2
- net ~{DTACK}: now also U21.19 (O)
- net ~{AS}: now reaches U21.10 (I)
- net ~{ROM_CS}: now reaches U21.14 (O)
- net ~{RAM_CS}: now reaches U21.15 (O)
- net ~{IO_CS}: now reaches U21.18 (O)
- net ~{BERR}: now reaches U21.20 (O)
- net HALT renamed ~{HALT}
- net IPL0 renamed ~{IPL0}
- net IPL1 renamed ~{IPL1}
- net IPL2 renamed ~{IPL2}
- net LDS renamed ~{LDS}
- net UDS renamed ~{UDS}
- net VPA renamed ~{VPA}
- new net ~{RESET}: R3.2, U1.18 (~{RESET}), U5.2
Other:
- moved on the sheet: C6, U21

Commit message: mega stuff
Parts:
- added C7: 100n, symbol Device:C
- added J1: PLD JTAG, 4ms_Connector:Pins_2x05_2.54mm_TH, symbol 4ms_Connector:Pins_02x05_P2.54mm_TH
- added U3: ATF1508ASx-xxJx84, Package_LCC:PLCC-84_29.3x29.3mm_P1.27mm, symbol CPLD_Microchip:ATF1508ASx-xxJx84
Connections:
- net +5V: now also C7.1, J1.4 (GND)
- net GND: now also C7.2, J1.10 (-12V), J1.2 (+12V), U3.19 (GND), U3.32 (GND), U3.42 (GND), U3.47 (GND), U3.59 (GND), U3.7 (GND), U3.72 (GND), U3.82 (GND)
- new net: U3.13 (VCCIO), U3.26 (VCCIO), U3.38 (VCCIO), U3.53 (VCCIO), U3.66 (VCCIO), U3.78 (VCCIO)
- new net: U3.3 (VCCINT), U3.43 (VCCINT)
- new net TCK: J1.1 (+12V), U3.62 (I/O/TCK)
- new net TDI: J1.9 (-12V), U3.14 (I/O/TDI)
- new net TDO: J1.3 (GND), U3.71 (I/O/TDO)
- new net TMS: J1.5 (GND), U3.23 (I/O/TMS)
- no-connect marks 0 -> 3
Other:
- moved on the sheet: C10, C11, C12, C13, C14, C15, C2, C3, C4, C5, C6, C8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

Commit message: mega stuff
Parts:
- removed C13, C14, C15, C6, C9: 100n, symbol Device:C
- removed U10, U9: AS6C4008-55PCN, Package_DIP:DIP-32_W15.24mm, symbol Memory_RAM:AS6C4008-55PCN
- removed U13, U14: SST39SF040, symbol Memory_Flash:SST39SF040
- removed U21: ATF22V10, Package_DIP:DIP-24_W7.62mm_Socket, symbol my:ATF22V10
Connections:
- net +5V: now also U3.13 (VCCIO), U3.26 (VCCIO), U3.3 (VCCINT), U3.38 (VCCIO), U3.43 (VCCINT), U3.53 (VCCIO), U3.66 (VCCIO), U3.78 (VCCIO)
- net A10: now also U3.28 (I/O)
- net A11: now also U3.27 (I/O)
- net A12: now also U3.25 (I/O)
- net A13: now also U3.24 (I/O)
- net A14: now also U3.22 (I/O)
- net A15: now also U3.21 (I/O)
- net A16: now also U3.20 (I/O)
- net A17: now also U3.18 (I/O)
- net A18: now also U3.17 (I/O)
- net A19: now also U3.16 (I/O)
- net A20: now also U3.15 (I/O)
- net A21: now also U3.12 (I/O/PD1)
- net A22: now also U3.11 (I/O)
- net A23: now also U3.10 (I/O)
- net A8: now also U3.30 (I/O)
- net A9: now also U3.29 (I/O)
- net MPUCLOCK: now also U3.4 (I/O)
- net RESET: now also U3.31 (I/O)
- net ~{AS}: now also U3.5 (I/O)
- net ~{BERR}: now also U3.81 (I/O/GCLK3)
- net ~{DTACK}: now also U3.80 (I/O)
- net ~{IO_CS}: now also U3.67 (I/O)
- net ~{LDS}: now also U3.9 (I/O)
- net ~{UDS}: now also U3.8 (I/O)
- net ~{RAML_OE}: now reaches U7.24 (OE#)
- net ~{RAML_OE}: now also U3.73 (I/O)
- net ~{RAML_WE}: now reaches U7.29 (WE#)
- net ~{RAML_WE}: now also U3.69 (I/O)
- net ~{RAMH_OE}: now reaches U8.24 (OE#)
- net ~{RAMH_OE}: now also U3.70 (I/O)
- net ~{RAMH_WE}: now reaches U8.29 (WE#)
- net ~{RAMH_WE}: now also U3.68 (I/O)
- net ~{VID_CS}: now reaches U3.57 (I/O)
- net ~{KBD_CS}: now reaches U3.58 (I/O)
- net R/W: now reaches U3.6 (I/O)
- net R/W: now also U1.9 (R/~{W})
- net ~{UART_CS}: now reaches U3.60 (I/O)
- net ~{IDE_DIOW}: now reaches U3.61 (I/O)
- net ~{IDE_DIOR}: now reaches U3.63 (I/O)
- net ~{IDE_CS1}: now reaches U3.64 (I/O)
- net ~{IDE_CS0}: now reaches U3.65 (I/O)
- net ~{RAMH_CS}: now reaches U3.74 (I/O)
- net ~{RAMH_CS}: now also U8.22 (CE#)
- net ~{RAML_CS}: now reaches U3.75 (I/O)
- net ~{RAML_CS}: now also U7.22 (CE#)
- net ~{ROM_OE}: now reaches U3.76 (I/O)
- net ~{ROMH_CS}: now reaches U3.77 (I/O)
- net ~{ROMH_CS}: now also U12.22 (CE)
- net ~{ROML_CS}: now reaches U3.79 (I/O)
- net ~{ROML_CS}: now also U11.22 (CE)
- removed net ~{RAM_CS}: U7.22 (CE#), U8.22 (CE#)
- removed net ~{ROM_CS}: U11.22 (CE), U12.22 (CE)
Other:
- moved on the sheet: C1, C7, J1, U1, U3
