File: pcb/misa.kicad_sch (KiCad schematic)
At the start: 41 parts, among them J1 PLD JTAG, J2 UART, J3 CF CARD, J4 44 PIN IDE, SW1 Reset, U1 MC68000P, U11 SST39SF040, U12 SST39SF040, U2 NE555P, U3 ATF1508ASx-xxJx84, U4 74HC74, U5 74LS05, U7 AS6C4008-55PCN, U8 AS6C4008-55PCN, U9 TL16C550DPTR, Y1 8MHz, Y2 1.8432MHz

Commit message: stuff
Parts:
- added unit 7 of U5
Connections:
- net +5V: now also U5.14 (VCC); no longer U5.14 (VCC)
- net GND: now also U5.7 (GND); no longer U5.7 (GND)
Other:
- moved on the sheet: C10, C11, C12, C4, C5, C8, U11, U12, U4C, U7, U8

Commit message: stuff
Parts:
- removed U9: TL16C550DPTR, TL16C550DPTR:QFP50P900X900X160-48N, symbol TL16C550DPTR:TL16C550DPTR
- added J1: DISPLAY, symbol Connector:Conn_01x20_Pin
- added U6: 16550, Package_DIP:DIP-40_W15.24mm, symbol Interface_UART:16550
- R7: renamed from R13; value 220R -> 470R
- renumbered C11 to C10, C12 to C11, C2 to C12, C3 to C13, C4 to C2, C5 to C3, C9 to C4, C13 to C5, C7 to C6, C6 to C7, C10 to C8, C8 to C9, J4 to J2, J2 to J4, J1 to J5, JP2 to JP1, JP3 to JP2, JP4 to JP3, R6 to R1, R5 to R2, R1 to R3, R3 to R4, R2 to R5, R4 to R6, U8 to U10, U5 to U2, U4 to U3, U3 to U4, U11 to U5, U2 to U8, U12 to U9, Y2 to Y1, Y1 to Y2
Connections:
- net +5V: now also J1.2 (Pin_2), U6.12 (CS0), U6.13 (CS1), U6.40 (VCC)
- net A1: now also J1.7 (Pin_7), U6.28 (A0)
- net A2: now also U6.27 (A1)
- net A3: now also U6.26 (A2)
- net D0: now also J1.9 (Pin_9), U6.1 (D0)
- net D1: now also J1.10 (Pin_10), U6.2 (D1)
- net D2: now also J1.11 (Pin_11), U6.3 (D2)
- net D3: now also J1.12 (Pin_12), U6.4 (D3)
- net D4: now also J1.13 (Pin_13), U6.5 (D4)
- net D5: now also J1.14 (Pin_14), U6.6 (D5)
- net D6: now also J1.15 (Pin_15), U6.7 (D6)
- net D7: now also J1.16 (Pin_16), U6.8 (D7)
- net GND: now also J1.1 (Pin_1), U6.19 (WR), U6.20 (GND), U6.22 (RD)
- net RESET: now also U2.5, U6.35 (MR)
- net UART_INTR: now also U6.30 (INTR)
- net ~{HALT}: no longer U2.5
- net ~{RESET}: now also J1.8 (Pin_8)
- net ~{UART_CS}: now also U6.14 (~{CS2})
- net ~{UART_RD}: now also U6.21 (~{RD})
- net ~{UART_WR}: now also U6.18 (~{WR})
- net ~{VID_CS}: now also J1.6 (Pin_6)
- net at Y1.5 (OUT): now also U6.16 (XIN)
- net ~{VID_WR}: now reaches U4.52 (I/O)
- net ~{VID_WR}: now also J1.4 (Pin_4)
- net ~{VID_RD}: now reaches U4.54 (I/O)
- net ~{VID_RD}: now also J1.5 (Pin_5)
- net SIN: no longer names the net of J4.2 (Pin_2)
- net SIN: now also U6.10 (SIN)
- net SOUT: no longer names the net of J4.3 (Pin_3)
- net SOUT: now also U6.11 (SOUT)
Other:
- note added: "DISPLAY 320240B RA8835A"
- moved on the sheet: C10, C11, C2, C3, C4, C5, C6, C7, C8, C9, D1, J2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

Commit message: wifi
Parts:
- added C14: 100n, symbol Device:C
- added R10, R8, R9: 10K, Resistor_THT:R_Axial_DIN0207_L6.3mm_D2.5mm_P7.62mm_Horizontal, symbol Device:R
- added U11: WizFi360, WizFi360:Untitled, symbol WizFi360:WizFi360
- U1: footprint Package_DIP:DIP-64_W22.86mm -> Package_LCC:PLCC-68_THT-Socket
- U4: footprint Package_LCC:PLCC-84_29.3x29.3mm_P1.27mm -> Package_LCC:PLCC-84_THT-Socket
- U5, U9: footprint (none) -> Package_LCC:PLCC-32_THT-Socket
- U6: footprint Package_DIP:DIP-40_W15.24mm -> Package_LCC:PLCC-44_THT-Socket
- Y1: value 1.8432MHz -> 1.8432 MHz
- Y2: value 8MHz -> 16 MHz
Connections:
- net GND: now also C14.2, R10.2, U11.15 (GND)
- net ~{RESET}: now also U11.1 (RST)
- new net: R10.1, U11.4 (WP)
- new net: R8.2, U11.3 (PA0)
- new net: R9.2, U11.5 (PA1)
- new net +3.3V: C14.1, R8.1, R9.1, U11.8 (VCC)
Other:
- note added: "WIFI"

Commit message: stuff
Parts:
- added C15, C16, C17: 100n, symbol Device:C
- added C18, C19: 3.3nF, symbol Device:C
- added R11: 100R, symbol Device:R
- added U12: YM2151, Package_DIP:DIP-24_18.0mmx34.29mm_W15.24mm_Socket_LongPads, symbol YM2151:YM2151
- added U13: YM3012, Package_DIP:DIP-16_W7.62mm_Socket_LongPads, symbol YM3012:YM3012
- added U14: TL074, symbol Amplifier_Operational:TL074
Connections:
- net +5V: now also C15.1, C16.1, C17.1, U12.22 (VDD), U13.1 (VDD), U14.4 (V+)
- net GND: now also C15.2, C16.2, C17.2, C18.2, C19.2, U12.1 (VSS), U12.11 (VSS), U13.16 (VSS_A), U13.3 (VSS_D), U13.8 (VSS_A), U14.11 (V-)
- net ~{RESET}: now also U12.3 (~{IC}), U13.7 (~{ICL})
- new net: C18.1, U13.9 (CH1), U14.10 (+)
- new net: C19.1, U13.10 (CH2), U14.12 (+)
- new net: R11.2, U13.11 (AIN)
- new net: U13.12 (AOUT), U14.5 (+)
- new net: U13.13 (MP), U14.1
- new net: U13.14 (BC), U14.2 (-)
- new net: U13.15 (RB), U14.3 (+)
- new net: U12.23 (o1), U13.2 (CLOCK)
- new net: U12.21 (SO), U13.4 (SD)
- new net: U12.19 (SH2), U13.5 (SAM2)
- new net: U12.20 (SH1), U13.6 (SAM1)
- new net: R11.1, U14.6 (-), U14.7
- new net AUD_CLOCK: U12.24 (oM)
- new net L_OUT: U14.8, U14.9 (-)
- new net R_OUT: U14.13 (-), U14.14
Other:
- note added: "AUDIO"
- moved on the sheet: C14, R10, R8, R9, U11

Commit message: stuff
Parts:
- removed R2: 10K, Resistor_THT:R_Axial_DIN0207_L6.3mm_D2.5mm_P7.62mm_Horizontal, symbol Device:R
- added Y3: 3.579545 MHz, Oscillator:Oscillator_DIP-8, symbol Oscillator:CXO_DIP8
Connections:
- net +5V: now also Y3.8 (Vcc)
- net GND: now also Y3.4 (GND)
- net AUD_CLOCK: no longer names the net of U12.24 (oM)
- net AUD_CLOCK: now also Y3.5 (OUT)
Other:
- moved on the sheet: C4, C5, J2, J3

Commit message: stuff
Parts:
- removed J1: DISPLAY, symbol Connector:Conn_01x20_Pin
- removed R1: 10K, Resistor_THT:R_Axial_DIN0207_L6.3mm_D2.5mm_P7.62mm_Horizontal, symbol Device:R
- added C19, C20: 100uF, Capacitor_THT:CP_Radial_D5.0mm_P2.50mm, symbol Device:C_Polarized
- added C21, C23, C24: 470uF, Capacitor_THT:CP_Radial_D6.3mm_P2.50mm, symbol Device:C_Polarized
- added C25, C26: 3.3nF, Capacitor_THT:C_Rect_L7.0mm_W2.5mm_P5.00mm, symbol Device:C
- added D2: 1N4148, Diode_THT:D_DO-35_SOD27_P7.62mm_Horizontal, symbol Diode:1N4148
- added J5: Headphones, Connector_Audio:Jack_6.35mm_Neutrik_NMJ6HFD2-AU_Horizontal, symbol Connector_Audio:AudioJack3_Dual_Switch
- added K1: G5V-2, Relay_THT:Relay_DPDT_Omron_G5V-2, symbol Relay:G5V-2
- added LS1, LS2: 8R 1W, Connector_PinHeader_2.54mm:PinHeader_1x02_P2.54mm_Vertical, symbol Device:Speaker
- added Q1: NPN, Package_TO_SOT_THT:TO-92L_Inline_Wide, symbol Simulation_SPICE:NPN
- added R10, R11: 10K, Resistor_THT:R_Axial_DIN0207_L6.3mm_D2.5mm_P7.62mm_Horizontal, symbol Device:R
- added R12, R13: 100R, Resistor_THT:R_Axial_DIN0207_L6.3mm_D2.5mm_P7.62mm_Horizontal, symbol Device:R
- added R14, R16: 33R, Resistor_THT:R_Axial_DIN0207_L6.3mm_D2.5mm_P7.62mm_Horizontal, symbol Device:R
- added R15, R17: 4.7R, Resistor_THT:R_Axial_DIN0207_L6.3mm_D2.5mm_P7.62mm_Horizontal, symbol Device:R
- added R9: 47K, Resistor_THT:R_Axial_DIN0207_L6.3mm_D2.5mm_P7.62mm_Horizontal, symbol Device:R
- added RV1: VOL, symbol GBVOL:GBVOL
- added RV2: Contrast, symbol Device:R_Potentiometer_Trim
- added U16: TDA2822M, Package_DIP:DIP-8_W7.62mm_Socket_LongPads, symbol TDA2822M:TDA2822M
- added U5: KNY320240B, KNY320240B:KNY320240B, symbol KNY320240B:KNY320240B
- added U8: 18650 Holder, 18650_holder:18650_holder, symbol 18650holder:18650holder
- C1: renamed from C12; footprint (none) -> Capacitor_THT:C_Rect_L7.0mm_W2.5mm_P5.00mm
- C11: renamed from C7; footprint (none) -> Capacitor_THT:C_Rect_L7.0mm_W2.5mm_P5.00mm
- C12: renamed from C5; footprint (none) -> Capacitor_THT:C_Rect_L7.0mm_W2.5mm_P5.00mm
- C13: renamed from C8; footprint (none) -> Capacitor_THT:C_Rect_L7.0mm_W2.5mm_P5.00mm
- C14: renamed from C10; footprint (none) -> Capacitor_THT:C_Rect_L7.0mm_W2.5mm_P5.00mm
- C15: renamed from C14; footprint (none) -> Capacitor_THT:C_Rect_L7.0mm_W2.5mm_P5.00mm
- C16: renamed from C9; footprint (none) -> Capacitor_THT:C_Rect_L7.0mm_W2.5mm_P5.00mm
- C17: renamed from C11; footprint (none) -> Capacitor_THT:C_Rect_L7.0mm_W2.5mm_P5.00mm
- C18: renamed from C15; footprint (none) -> Capacitor_THT:C_Rect_L7.0mm_W2.5mm_P5.00mm
- C2: renamed from C1; footprint (none) -> Capacitor_THT:C_Rect_L7.0mm_W2.5mm_P5.00mm
- C22: renamed from C16; footprint (none) -> Capacitor_THT:C_Rect_L7.0mm_W2.5mm_P5.00mm
- C27: renamed from C18; footprint (none) -> Capacitor_THT:C_Rect_L7.0mm_W2.5mm_P5.00mm
- C28: renamed from C19; footprint (none) -> Capacitor_THT:C_Rect_L7.0mm_W2.5mm_P5.00mm
- C3: renamed from C6; footprint (none) -> Capacitor_THT:C_Rect_L7.0mm_W2.5mm_P5.00mm
- C4: renamed from C13; footprint (none) -> Capacitor_THT:CP_Radial_D4.0mm_P2.00mm
- C5: renamed from C2; footprint (none) -> Capacitor_THT:C_Rect_L7.0mm_W2.5mm_P5.00mm
- C6: renamed from C3; footprint (none) -> Capacitor_THT:C_Rect_L7.0mm_W2.5mm_P5.00mm
- C7: renamed from C17; footprint (none) -> Capacitor_THT:C_Rect_L7.0mm_W2.5mm_P5.00mm
- C8: renamed from C4; footprint (none) -> Capacitor_THT:C_Rect_L7.0mm_W2.5mm_P5.00mm
- D1: footprint (none) -> LED_THT:LED_D3.0mm
- R18: renamed from R11; footprint (none) -> Resistor_THT:R_Axial_DIN0207_L6.3mm_D2.5mm_P7.62mm_Horizontal
- U4: renamed from U2; footprint (none) -> Package_DIP:DIP-14_W7.62mm_Socket_LongPads
- U6: renamed from U3; footprint (none) -> Package_DIP:DIP-14_W7.62mm_Socket_LongPads
- U7: renamed from U14; footprint (none) -> Package_DIP:DIP-14_W7.62mm_Socket_LongPads
- renumbered J5 to J1, J3 to J2, J2 to J3, R3 to R1, R5 to R2, R4 to R3, R6 to R4, R7 to R5, R9 to R6, R10 to R7, U5 to U10, U9 to U11, U11 to U12, U7 to U13, U10 to U14, U12 to U15, U13 to U17, U4 to U2, U8 to U3, U6 to U9, Y2 to Y1, Y1 to Y2
Connections:
- net +3.3V: now also U8.11 (3V), U8.13 (3V), U8.15 (3V), U8.17 (3V), U8.19 (3V)
- net +5V: now also C21.1, R9.1, U16.2 (V+), U5.19 (LED+), U5.2 (VDD), U8.1 (5V), U8.3 (5V), U8.5 (5V), U8.7 (5V), U8.9 (5V)
- net A1: now also U15.4 (A0), U5.7 (A0)
- net D0: now also U15.10 (D0), U5.9 (D0)
- net D1: now also U15.12 (D1), U5.10 (D1)
- net D2: now also U15.13 (D2), U5.11 (D2)
- net D3: now also U15.14 (D3), U5.12 (D3)
- net D4: now also U15.15 (D4), U5.13 (D4)
- net D5: now also U15.16 (D5), U5.14 (D5)
- net D6: now also U15.17 (D6), U5.15 (D6)
- net D7: now also U15.18 (D7), U5.16 (D7)
- net GND: now also C19.2, C20.2, C21.2, D2.2 (A), J5.S1, K1.1, LS1.2, LS2.2, Q1.3 (E), R10.2, R11.2, R14.2, R15.2, R16.2, R17.2, RV1.1, RV1.MP, RV2.3, U16.4 (GND), U5.1 (VSS), U5.20 (LED-), U8.10 (GND), U8.12 (GND), U8.14 (GND), U8.16 (GND), U8.18 (GND), U8.2 (GND), U8.20 (GND), U8.4 (GND), U8.6 (GND), U8.8 (GND)
- net ~{RESET}: now also U5.8 (RES)
- net ~{VID_CS}: now also U5.6 (CS)
- net ~{VID_RD}: now also U5.5 (RD)
- net ~{VID_WR}: now also U5.4 (WR)
- net ~{AUDIO_RD}: now reaches U2.48 (I/O)
- net ~{AUDIO_RD}: now also U15.6 (RD)
- net ~{AUDIO_WR}: now reaches U2.49 (I/O)
- net ~{AUDIO_WR}: now also U15.5 (~{WR})
- net ~{AUDIO_CS}: now reaches U2.50 (I/O)
- net ~{AUDIO_CS}: now also U15.7 (~{CS})
- net ~{WIFI_CS}: now reaches U2.51 (I/O)
- net L_OUT renamed AMP_L
- net AMP_L: now also RV1.4
- net R_OUT renamed AMP_R
- net AMP_R: now also RV1.5
- new net: K1.11, LS2.1
- new net: J5.R1, R13.2, R14.1
- new net: R11.1, RV1.2, U16.6 (IN2+)
- new net: C23.1, U16.1 (OUT1)
- new net: C24.1, U16.3 (OUT2)
- new net: C20.1, U16.5 (IN2-)
- new net: R10.1, RV1.3, U16.7 (IN1+)
- new net: C19.1, U16.8 (IN1-)
- new net: D2.1 (K), K1.16, Q1.1 (C)
- new net: K1.6, LS1.1
- new net: RV2.1, U5.18 (VEE)
- new net: RV2.2, U5.3 (VO)
- new net: C25.2, R15.1
- new net: J5.T1, R12.2, R16.1
- new net: C26.2, R17.1
- new net HP_L: K1.8, R12.1
- new net HP_R: K1.9, R13.1
- new net HP_SW: J5.SN1, Q1.2 (B), R9.2
- new net OUT_L: C23.2, C26.1, K1.4
- new net OUT_R: C24.2, C25.1, K1.13
Other:
- moved on the sheet: C12, C15, C18, C22, C27, C28, C5, C6, C7, C8, J2, J3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

Commit message: stuff
Parts:
- added U18: 68681, symbol Interface:68681
Other:
- moved on the sheet: C11, J4, U9, Y2

Commit message: stuff
Parts:
- removed U9: 16550, Package_LCC:PLCC-44_THT-Socket, symbol Interface_UART:16550
- removed Y2: 1.8432 MHz, Oscillator:Oscillator_DIP-8, symbol Oscillator:CXO_DIP8
Connections:
- net +5V: now also U18.40 (VCC)
- net A1: now also U18.1 (RS1)
- net A2: now also U18.3 (RS2)
- net A3: now also U18.5 (RS3)
- net A4: now also U18.6 (RS4)
- net D0: now also U18.25 (D0)
- net D1: now also U18.16 (D1)
- net D2: now also U18.24 (D2)
- net D3: now also U18.17 (D3)
- net D4: now also U18.23 (D4)
- net D5: now also U18.18 (D5)
- net D6: now also U18.22 (D6)
- net D7: now also U18.19 (D7)
- net GND: now also U18.20 (GND)
- net at U18.30 (TXDA): now also J4.2 (Pin_2)
- net at U18.31 (RXDA): now also J4.3 (Pin_3)
- no-connect marks 20 -> 12
Other:
- moved on the sheet: C11, J4, U18
