File: pcb/misa.kicad_sch (KiCad schematic)
At the start: 80 parts, among them J1 PLD JTAG, J2 CF CARD, J3 44 PIN IDE, J4 UART, J5 Headphones, K1 G5V-2, Q1 NPN, SW1 Reset, U1 MC68000P, U10 SST39SF040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

Commit message: stuff
Parts:
- added C10, C9: 20p, symbol Device:C
- added Y2: Crystal, symbol Device:Crystal
Connections:
- net GND: now also C10.2, C9.2
- net at U18.32 (X1/CLK): now also C9.1, Y2.1
- net at U18.33 (X2): now also C10.1, Y2.2
Other:
- note added: "DUART"
- note removed: "UART"

Commit message: stuff
Parts:
- Y2: value Crystal -> 3.6864 MHz
Connections:
- net GND: now also C10.1; no longer C10.2
- net ~{RESET}: now also U18.34 (RESET)
- net ~{UART_CS}: now also U18.35 (CS)
- net at U18.33 (X2), Y2.2: now also C10.2; no longer C10.1
Other:
- moved on the sheet: C10, Y2

Commit message: stuff
Parts:
- removed J4: UART, 4ms_Connector:Pins_1x04_2.54mm_TH_SWD, symbol 4ms_Connector:Conn_01x04
- added J6: EXT_CLOCK, symbol Connector:Conn_01x01_Pin
- added J7: Conn_01x06, 4ms_Connector:Pins_1x06_2.54mm_TH_SWD, symbol 4ms_Connector:Conn_01x06
- added JP4: Jumper_2_Open, Connector_PinHeader_2.54mm:PinHeader_1x02_P2.54mm_Vertical, symbol Jumper:Jumper_2_Open
Connections:
- net +5V: now also J7.1 (Pin_1)
- net GND: now also J7.2 (Pin_2)
- net MPUCLOCK: now also JP4.2 (B)
- net at U18.29 (OP0): now also J7.5 (Pin_5)
- net at U18.30 (TXDA): now also J7.3 (Pin_3)
- net at U18.31 (RXDA): now also J7.4 (Pin_4)
- net at U18.7 (IP0): now also J7.6 (Pin_6)
- new net: J6.1 (Pin_1), JP4.1 (A)
Other:
- moved on the sheet: C12, C15, C5, C6, C7, C8, J2, J3, JP1, JP2, JP3, R6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
