File: pcb/misa.kicad_pcb (KiCad board)
At the start: 2 copper layers, 12 parts, among them J1 PLD JTAG, J2 UART, J3 CF CARD, U1 MC68000P, U2 NE555P, U3 ATF1508ASx-xxJx84, U6 16550, U7 AS6C4008-55PCN, U8 AS6C4008-55PCN, U9 TL16C550DPTR, Y1 8MHz, Y2 1.8432MHz

Commit message: wifi
Parts:
- removed J1: PLD JTAG, 4ms_Connector:Pins_2x05_2.54mm_TH
- removed U2: NE555P, Package_DIP:DIP-8_W7.62mm
- removed U3: ATF1508ASx-xxJx84, Package_QFP:TQFP-100-1EP_14x14mm_P0.5mm_EP5x5mm
- added J4: UART, 4ms_Connector:Pins_1x04_2.54mm_TH_SWD, F.Cu at (93.5, 20.5)
- added J5: PLD JTAG, 4ms_Connector:Pins_2x05_2.54mm_TH, F.Cu at (193.5, 83.5)
- added JP1: Jumper_2_Open, Connector_PinHeader_2.54mm:PinHeader_1x02_P2.54mm_Vertical, F.Cu at (164.7, 36.6)
- added JP2: Jumper_2_Open, Connector_PinHeader_2.54mm:PinHeader_1x02_P2.54mm_Vertical, F.Cu at (169.2, 36.6)
- added JP3: Jumper_2_Open, Connector_PinHeader_2.54mm:PinHeader_1x02_P2.54mm_Vertical, F.Cu at (173.8, 36.6)
- added R1: 10K, Resistor_THT:R_Axial_DIN0207_L6.3mm_D2.5mm_P7.62mm_Horizontal, F.Cu at (128.8, 113.0)
- added R10: 10K, Resistor_THT:R_Axial_DIN0207_L6.3mm_D2.5mm_P7.62mm_Horizontal, F.Cu at (253.4, 95.5)
- added R2: 10K, Resistor_THT:R_Axial_DIN0207_L6.3mm_D2.5mm_P7.62mm_Horizontal, F.Cu at (128.8, 117.0)
- added R3: 1M, Resistor_THT:R_Axial_DIN0207_L6.3mm_D2.5mm_P7.62mm_Horizontal, F.Cu at (128.8, 121.1)
- added R4: 10K, Resistor_THT:R_Axial_DIN0207_L6.3mm_D2.5mm_P7.62mm_Horizontal, F.Cu at (128.8, 125.2)
- added R5: 1M, Resistor_THT:R_Axial_DIN0207_L6.3mm_D2.5mm_P7.62mm_Horizontal, F.Cu at (128.8, 129.2)
- added R6: 10K, Resistor_THT:R_Axial_DIN0207_L6.3mm_D2.5mm_P7.62mm_Horizontal, F.Cu at (128.8, 133.2)
- added R7: 470R, Resistor_THT:R_Axial_DIN0207_L6.3mm_D2.5mm_P7.62mm_Horizontal, F.Cu at (128.8, 137.3)
- added R8: 10K, Resistor_THT:R_Axial_DIN0207_L6.3mm_D2.5mm_P7.62mm_Horizontal, F.Cu at (253.4, 87.4)
- added R9: 10K, Resistor_THT:R_Axial_DIN0207_L6.3mm_D2.5mm_P7.62mm_Horizontal, F.Cu at (253.4, 91.5)
- added U10: AS6C4008-55PCN, Package_DIP:DIP-32_W15.24mm, F.Cu at (133.0, 70.8)
- added U11: WizFi360, WizFi360:Untitled, F.Cu at (241.9, 94.4)
- added U4: ATF1508ASx-xxJx84, Package_LCC:PLCC-84_THT-Socket, F.Cu at (168.8, 72.5)
- added U5: SST39SF040, Package_LCC:PLCC-32_THT-Socket, F.Cu at (194.8, 45.5)
- J2: value UART -> 44 PIN IDE; footprint 4ms_Connector:Pins_1x04_2.54mm_TH_SWD -> Connector_PinSocket_2.54mm:PinSocket_2x22_P2.54mm_Vertical
- U1: footprint Package_DIP:DIP-64_W22.86mm -> Package_LCC:PLCC-68_THT-Socket
- U6: footprint Package_DIP:DIP-40_W15.24mm -> Package_LCC:PLCC-44_THT-Socket
- U8: value AS6C4008-55PCN -> NE555P; footprint Package_DIP:DIP-32_W15.24mm -> Package_DIP:DIP-8_W7.62mm
- U9: value TL16C550DPTR -> SST39SF040; footprint TL16C550DPTR:QFP50P900X900X160-48N -> Package_LCC:PLCC-32_THT-Socket
- Y1: value 8MHz -> 1.8432 MHz
- Y2: value 1.8432MHz -> 16 MHz
- moved J2 127.2 mm to (92.3, 36.7)
- moved U6 113.0 mm to (61.0, 34.0)
- moved U1 88.5 mm to (166.3, 110.6)
- moved U9 76.2 mm to (215.0, 45.5)
- moved Y1 63.2 mm to (116.3, 121.9)
- moved Y2 63.2 mm to (116.3, 136.2)
- moved U8 57.0 mm to (163.9, 43.5)
- moved U7 24.1 mm to (114.6, 70.8)
- moved J3 24.1 mm to (137.7, 43.8)
Connections:
- J2 pad 1: +5V -> ~{RESET}
- J2 pad 2: SIN -> GND
- J2 pad 3: SOUT -> D7
- J2 pad 4: GND -> D8
- U8 pad 1: A19 -> GND
- U8 pad 2: A17 -> Net-(U8-TR)
- U8 pad 3: A15 -> RESET
- U8 pad 4: A13 -> +5V
- U8 pad 5: A8 -> GND
- U8 pad 6: A7 -> Net-(U8-DIS)
- U8 pad 7: A6 -> Net-(U8-DIS)
- U8 pad 8: A5 -> +5V
- U9 pad 1: (no net) -> A19
- U9 pad 10: +5V -> A3
- U9 pad 11: ~{UART_CS} -> A2
- U9 pad 12: unconnected-(U9-~{BAUDOUT}-Pad12) -> A1
- U9 pad 13: (no net) -> D8
- U9 pad 14: Net-(U9-XIN) -> D9
- U9 pad 15: unconnected-(U9-XOUT-Pad15) -> D10
- U9 pad 16: ~{UART_WR} -> GND
- U9 pad 17: GND -> D11
- U9 pad 18: GND -> D12
- U9 pad 19: ~{UART_RD} -> D13
- U9 pad 2: D5 -> A17
- U9 pad 20: GND -> D14
- U9 pad 21: (no net) -> D15
- U9 pad 22: unconnected-(U9-DDIS-Pad22) -> ~{ROMH_CS}
- U9 pad 23: unconnected-(U9-~{TXRDY}-Pad23) -> A11
- U9 pad 25: (no net) -> A12
- U9 pad 26: A3 -> A10
- U9 pad 27: A2 -> A9
- U9 pad 28: A1 -> A14
- U9 pad 29: unconnected-(U9-~{RXRDY}-Pad29) -> A15
- U9 pad 3: D6 -> A16
- U9 pad 30: UART_INTR -> A18
- U9 pad 32: unconnected-(U9-~{RTS}-Pad32) -> +5V
- U9 pad 4: D7 -> A13
- U9 pad 5: unconnected-(U9-RCLK-Pad5) -> A8
- U9 pad 6: (no net) -> A7
- U9 pad 7: SIN -> A6
- U9 pad 8: SOUT -> A5
- U9 pad 9: +5V -> A4
- Y1 pad 5: 1/1CLOCK -> Net-(U6-XIN)
- Y2 pad 5: Net-(U9-XIN) -> 1/1CLOCK

Commit message: stuff
Parts:
- added C1: 100n, Capacitor_THT:C_Rect_L7.0mm_W2.5mm_P5.00mm, F.Cu at (272.2, 141.6)
- added C11: 100n, Capacitor_THT:C_Rect_L7.0mm_W2.5mm_P5.00mm, F.Cu at (280.8, 141.6)
- added C12: 100n, Capacitor_THT:C_Rect_L7.0mm_W2.5mm_P5.00mm, F.Cu at (280.8, 145.6)
- added C13: 100n, Capacitor_THT:C_Rect_L7.0mm_W2.5mm_P5.00mm, F.Cu at (280.8, 149.7)
- added C14: 100n, Capacitor_THT:C_Rect_L7.0mm_W2.5mm_P5.00mm, F.Cu at (280.8, 153.7)
- added C15: 100n, Capacitor_THT:C_Rect_L7.0mm_W2.5mm_P5.00mm, F.Cu at (280.8, 157.8)
- added C16: 100n, Capacitor_THT:C_Rect_L7.0mm_W2.5mm_P5.00mm, F.Cu at (280.8, 161.8)
- added C17: 100n, Capacitor_THT:C_Rect_L7.0mm_W2.5mm_P5.00mm, F.Cu at (280.8, 165.9)
- added C18: 100n, Capacitor_THT:C_Rect_L7.0mm_W2.5mm_P5.00mm, F.Cu at (289.3, 141.6)
- added C19: 100uF, Capacitor_THT:CP_Radial_D5.0mm_P2.50mm, F.Cu at (320.5, 231.6)
- added C2: 100n, Capacitor_THT:C_Rect_L7.0mm_W2.5mm_P5.00mm, F.Cu at (272.2, 145.6)
- added C20: 100uF, Capacitor_THT:CP_Radial_D5.0mm_P2.50mm, F.Cu at (320.5, 238.1)
- added C21: 470uF, Capacitor_THT:CP_Radial_D6.3mm_P2.50mm, F.Cu at (324.4, 143.5)
- added C22: 100n, Capacitor_THT:C_Rect_L7.0mm_W2.5mm_P5.00mm, F.Cu at (289.3, 145.6)
- added C23: 470uF, Capacitor_THT:CP_Radial_D6.3mm_P2.50mm, F.Cu at (324.4, 151.3)
- added C24: 470uF, Capacitor_THT:CP_Radial_D6.3mm_P2.50mm, F.Cu at (324.4, 159.2)
- added C25: 3.3nF, Capacitor_THT:C_Rect_L7.0mm_W2.5mm_P5.00mm, F.Cu at (289.3, 149.7)
- added C26: 3.3nF, Capacitor_THT:C_Rect_L7.0mm_W2.5mm_P5.00mm, F.Cu at (289.3, 153.7)
- added C27: 3.3nF, Capacitor_THT:C_Rect_L7.0mm_W2.5mm_P5.00mm, F.Cu at (289.3, 157.8)
- added C28: 3.3nF, Capacitor_THT:C_Rect_L7.0mm_W2.5mm_P5.00mm, F.Cu at (289.3, 161.8)
- added C3: 100n, Capacitor_THT:C_Rect_L7.0mm_W2.5mm_P5.00mm, F.Cu at (272.2, 149.7)
- added C4: 1u, Capacitor_THT:CP_Radial_D4.0mm_P2.00mm, F.Cu at (325.1, 84.4)
- added C5: 100n, Capacitor_THT:C_Rect_L7.0mm_W2.5mm_P5.00mm, F.Cu at (272.2, 153.7)
- added C6: 100n, Capacitor_THT:C_Rect_L7.0mm_W2.5mm_P5.00mm, F.Cu at (272.2, 157.8)
- added C7: 100n, Capacitor_THT:C_Rect_L7.0mm_W2.5mm_P5.00mm, F.Cu at (272.2, 161.8)
- added C8: 100n, Capacitor_THT:C_Rect_L7.0mm_W2.5mm_P5.00mm, F.Cu at (272.2, 165.9)
- added D1: RUN, LED_THT:LED_D3.0mm, F.Cu at (290.6, 237.8)
- added D2: 1N4148, Diode_THT:D_DO-35_SOD27_P7.62mm_Horizontal, F.Cu at (282.4, 233.3)
- added J1: PLD JTAG, 4ms_Connector:Pins_2x05_2.54mm_TH, F.Cu at (326.7, 74.3)
- added K1: G5V-2, Relay_THT:Relay_DPDT_Omron_G5V-2, F.Cu at (313.6, 69.2)
- added LS1: 8R 1W, Connector_PinHeader_2.54mm:PinHeader_1x02_P2.54mm_Vertical, F.Cu at (273.9, 233.8)
- added LS2: 8R 1W, Connector_PinHeader_2.54mm:PinHeader_1x02_P2.54mm_Vertical, F.Cu at (278.5, 233.8)
- added Q1: NPN, Package_TO_SOT_THT:TO-92L_Inline_Wide, F.Cu at (282.3, 238.3)
- added R11: 10K, Resistor_THT:R_Axial_DIN0207_L6.3mm_D2.5mm_P7.62mm_Horizontal, F.Cu at (302.5, 130.1)
- added R12: 100R, Resistor_THT:R_Axial_DIN0207_L6.3mm_D2.5mm_P7.62mm_Horizontal, F.Cu at (302.5, 134.1)
- added R13: 100R, Resistor_THT:R_Axial_DIN0207_L6.3mm_D2.5mm_P7.62mm_Horizontal, F.Cu at (313.2, 113.9)
- added R14: 33R, Resistor_THT:R_Axial_DIN0207_L6.3mm_D2.5mm_P7.62mm_Horizontal, F.Cu at (313.2, 117.9)
- added R15: 4.7R, Resistor_THT:R_Axial_DIN0207_L6.3mm_D2.5mm_P7.62mm_Horizontal, F.Cu at (313.2, 122.0)
- added R16: 33R, Resistor_THT:R_Axial_DIN0207_L6.3mm_D2.5mm_P7.62mm_Horizontal, F.Cu at (313.2, 126.0)
- added R17: 4.7R, Resistor_THT:R_Axial_DIN0207_L6.3mm_D2.5mm_P7.62mm_Horizontal, F.Cu at (313.2, 130.1)
- added R18: 100R, Resistor_THT:R_Axial_DIN0207_L6.3mm_D2.5mm_P7.62mm_Horizontal, F.Cu at (313.2, 134.1)
- added U12: WizFi360, WizFi360:Untitled, F.Cu at (231.0, 225.2)
- added U13: AS6C4008-55PCN, Package_DIP:DIP-32_W15.24mm, F.Cu at (222.6, 176.0)
- added U14: AS6C4008-55PCN, Package_DIP:DIP-32_W15.24mm, F.Cu at (241.0, 176.0)
- added U15: YM2151, Package_DIP:DIP-24_18.0mmx34.29mm_W15.24mm_Socket_LongPads, F.Cu at (313.7, 35.2)
- added U16: TDA2822M, Package_DIP:DIP-8_W7.62mm_Socket_LongPads, F.Cu at (297.9, 230.4)
- added U17: YM3012, Package_DIP:DIP-16_W7.62mm_Socket_LongPads, F.Cu at (243.0, 218.3)
- added U2: ATF1508ASx-xxJx84, Package_LCC:PLCC-84_THT-Socket, F.Cu at (276.9, 177.8)
- added U3: NE555P, Package_DIP:DIP-8_W7.62mm, F.Cu at (309.2, 230.3)
- added Y3: 3.579545 MHz, Oscillator:Oscillator_DIP-8, F.Cu at (300.6, 70.7)
- J2: value 44 PIN IDE -> CF CARD; footprint Connector_PinSocket_2.54mm:PinSocket_2x22_P2.54mm_Vertical -> rc-cfcard:CF_Card_Socket_PTH; moved to B.Cu
- J3: value CF CARD -> 44 PIN IDE; footprint rc-cfcard:CF_Card_Socket_PTH -> Connector_PinSocket_2.54mm:PinSocket_2x22_P2.54mm_Vertical
- J5: value PLD JTAG -> Headphones; footprint 4ms_Connector:Pins_2x05_2.54mm_TH -> Connector_Audio:Jack_6.35mm_Neutrik_NMJ6HFD2-AU_Horizontal
- R1, R2: value 10K -> 1M
- R3: value 1M -> 10K
- R5: value 1M -> 470R
- R7: value 470R -> 10K
- R9: value 10K -> 47K
- U10: value AS6C4008-55PCN -> SST39SF040; footprint Package_DIP:DIP-32_W15.24mm -> Package_LCC:PLCC-32_THT-Socket
- U11: value WizFi360 -> SST39SF040; footprint WizFi360:Untitled -> Package_LCC:PLCC-32_THT-Socket
- U4: value ATF1508ASx-xxJx84 -> 74LS05; footprint Package_LCC:PLCC-84_THT-Socket -> Package_DIP:DIP-14_W7.62mm_Socket_LongPads
- U5: value SST39SF040 -> KNY320240B; footprint Package_LCC:PLCC-32_THT-Socket -> KNY320240B:KNY320240B
- U6: value 16550 -> 74HC74; footprint Package_LCC:PLCC-44_THT-Socket -> Package_DIP:DIP-14_W7.62mm_Socket_LongPads
- U7: value AS6C4008-55PCN -> TL074; footprint Package_DIP:DIP-32_W15.24mm -> Package_DIP:DIP-14_W7.62mm_Socket_LongPads
- U8: value NE555P -> 18650 Holder; footprint Package_DIP:DIP-8_W7.62mm -> 18650_holder:18650_holder; moved to B.Cu
- U9: value SST39SF040 -> 16550; footprint Package_LCC:PLCC-32_THT-Socket -> Package_LCC:PLCC-44_THT-Socket
- Y1: value 1.8432 MHz -> 16 MHz
- Y2: value 16 MHz -> 1.8432 MHz
- moved J4 316.4 mm to (327.0, 234.0)
- moved U6 277.1 mm to (271.6, 214.1)
- moved U8 269.6 mm to (427.4, 100.5), turned to 180 degrees
- moved U7 221.4 mm to (283.3, 214.1)
- moved JP1 219.0 mm to (260.1, 233.8)
- moved JP2 219.0 mm to (264.7, 233.8)
- moved JP3 219.0 mm to (269.3, 233.8)
- moved Y1 200.8 mm to (300.6, 42.2)
- moved Y2 200.8 mm to (300.6, 56.4)
- moved R7 175.2 mm to (302.5, 113.9)
- moved U10 170.3 mm to (301.4, 95.5)
- moved U4 168.4 mm to (259.9, 214.1)
- moved J5 167.5 mm to (303.9, 209.6)
- moved R1 162.9 mm to (291.7, 113.9)
- moved R2 162.9 mm to (291.7, 117.9)
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Connections:
- J2 pad 1: ~{RESET} -> GND
- J2 pad 10: D11 -> GND
- J2 pad 11: D3 -> GND
- J2 pad 12: D12 -> GND
- J2 pad 13: D2 -> +5V
- J2 pad 14: D13 -> GND
- J2 pad 15: D1 -> GND
- J2 pad 16: D14 -> GND
- J2 pad 17: D0 -> GND
- J2 pad 18: D15 -> A3
- J2 pad 19: GND -> A2
- J2 pad 2: GND -> D3
- J2 pad 20: unconnected-(J2-Pin_20-Pad20) -> A1
- J2 pad 21: unconnected-(J2-Pin_21-Pad21) -> D0
- J2 pad 22: GND -> D1
- J2 pad 23: ~{IDE_IOWR} -> D2
- J2 pad 24: GND -> unconnected-(J2-Pin_24-Pad24)
- J2 pad 25: ~{IDE_IORD} -> unconnected-(J2-Pin_25-Pad25)
- J2 pad 26: GND -> unconnected-(J2-Pin_26-Pad26)
- J2 pad 27: unconnected-(J2-Pin_27-Pad27) -> D11
- J2 pad 28: unconnected-(J2-Pin_28-Pad28) -> D12
- J2 pad 29: unconnected-(J2-Pin_29-Pad29) -> D13
- J2 pad 3: D7 -> D4
- J2 pad 30: GND -> D14
- J2 pad 31: unconnected-(J2-Pin_31-Pad31) -> D15
- J2 pad 32: unconnected-(J2-Pin_32-Pad32) -> ~{IDE_CS1}
- J2 pad 33: A2 -> GND
- J2 pad 34: unconnected-(J2-Pin_34-Pad34) -> ~{IDE_IORD}
- J2 pad 35: A1 -> ~{IDE_IOWR}
- J2 pad 36: A3 -> unconnected-(J2-Pin_36-Pad36)
- J2 pad 37: ~{IDE_CS0} -> unconnected-(J2-Pin_37-Pad37)
- J2 pad 38: ~{IDE_CS1} -> +5V
- J2 pad 39: unconnected-(J2-Pin_39-Pad39) -> GND
- J2 pad 4: D8 -> D5
- J2 pad 40: GND -> unconnected-(J2-Pin_40-Pad40)
- J2 pad 41: +5V -> ~{RESET}
- J2 pad 42: +5V -> unconnected-(J2-Pin_42-Pad42)
- J2 pad 43: GND -> unconnected-(J2-Pin_43-Pad43)
- J2 pad 6: D9 -> D7
- J2 pad 7: D5 -> ~{IDE_CS0}
- J2 pad 8: D10 -> GND
- J2 pad 9: D4 -> GND
- J3 pad 1: GND -> ~{RESET}
- J3 pad 10: GND -> D11
- J3 pad 11: GND -> D3
- J3 pad 12: GND -> D12
- J3 pad 13: +5V -> D2
- J3 pad 14: GND -> D13
- J3 pad 15: GND -> D1
- J3 pad 16: GND -> D14
- J3 pad 17: GND -> D0
- J3 pad 18: A3 -> D15
- J3 pad 19: A2 -> GND
- J3 pad 2: D3 -> GND
- J3 pad 20: A1 -> unconnected-(J3-Pin_20-Pad20)
- J3 pad 21: D0 -> unconnected-(J3-Pin_21-Pad21)
- J3 pad 22: D1 -> GND
- J3 pad 23: D2 -> ~{IDE_IOWR}
- J3 pad 24: unconnected-(J3-Pin_24-Pad24) -> GND
- J3 pad 25: unconnected-(J3-Pin_25-Pad25) -> ~{IDE_IORD}
- J3 pad 26: unconnected-(J3-Pin_26-Pad26) -> GND
- J3 pad 27: D11 -> unconnected-(J3-Pin_27-Pad27)
- J3 pad 28: D12 -> unconnected-(J3-Pin_28-Pad28)
- J3 pad 29: D13 -> unconnected-(J3-Pin_29-Pad29)
- J3 pad 3: D4 -> D7
- J3 pad 30: D14 -> GND
- J3 pad 31: D15 -> unconnected-(J3-Pin_31-Pad31)
- J3 pad 32: ~{IDE_CS1} -> unconnected-(J3-Pin_32-Pad32)
- J3 pad 33: GND -> A2
- J3 pad 34: ~{IDE_IORD} -> unconnected-(J3-Pin_34-Pad34)
- J3 pad 35: ~{IDE_IOWR} -> A1
- J3 pad 36: unconnected-(J3-Pin_36-Pad36) -> A3
- J3 pad 37: unconnected-(J3-Pin_37-Pad37) -> ~{IDE_CS0}
- J3 pad 38: +5V -> ~{IDE_CS1}
- J3 pad 39: GND -> unconnected-(J3-Pin_39-Pad39)
- J3 pad 4: D5 -> D8
- J3 pad 40: unconnected-(J3-Pin_40-Pad40) -> GND
- J3 pad 41: ~{RESET} -> +5V
- J3 pad 42: unconnected-(J3-Pin_42-Pad42) -> +5V
- J3 pad 43: unconnected-(J3-Pin_43-Pad43) -> GND
- J3 pad 6: D7 -> D9
- J3 pad 7: ~{IDE_CS0} -> D5
- J3 pad 8: GND -> D10
- J3 pad 9: GND -> D4
- R1 pad 2: Net-(Y1-EN) -> Net-(U3-TR)
- R10 pad 1: Net-(U11-WP) -> Net-(U16-IN1+)
- R2 pad 1: +5V -> Net-(U3-DIS)
- R2 pad 2: Net-(Y2-EN) -> +5V
- R3 pad 2: Net-(U8-TR) -> ~{RESET}
- R4 pad 2: ~{RESET} -> ~{HALT}
- R5 pad 1: Net-(U8-DIS) -> Net-(R5-Pad1)
- R5 pad 2: +5V -> Net-(D1-K)
- R6 pad 1: +5V -> +3.3V
- R6 pad 2: ~{HALT} -> Net-(U12-PA1)
- R7 pad 2: Net-(D1-K) -> GND
- R8 pad 2: Net-(U11-PA0) -> Net-(U12-PA0)
- R9 pad 1: +3.3V -> +5V
- R9 pad 2: Net-(U11-PA1) -> HP_SW
- U10 pad 13: D8 -> D0
- U10 pad 14: D9 -> D1
- U10 pad 15: D10 -> D2
- U10 pad 17: D11 -> D3
- U10 pad 18: D12 -> D4
- U10 pad 19: D13 -> D5
- U10 pad 20: D14 -> D6
- U10 pad 21: D15 -> D7
- U10 pad 22: ~{RAMH_CS} -> ~{ROML_CS}
- U10 pad 24: ~{RAMH_OE} -> unconnected-(U10-OE-Pad24)
- U10 pad 29: ~{RAMH_WE} -> A15
- U10 pad 3: A15 -> A16
- U10 pad 31: A16 -> unconnected-(U10-PGM-Pad31)
- U11 pad 1: ~{RESET} -> A19
- U11 pad 10: unconnected-(U11-PB18-Pad10) -> A3
- U11 pad 11: unconnected-(U11-PB13-Pad11) -> A2
- U11 pad 12: unconnected-(U11-PB14-Pad12) -> A1
- U11 pad 13: unconnected-(U11-PB17-Pad13) -> D8
- U11 pad 14: unconnected-(U11-PB16-Pad14) -> D9
- U11 pad 15: GND -> D10
- U11 pad 16: unconnected-(U11-PB10-Pad16) -> GND
- U11 pad 17: unconnected-(U11-TXD0-Pad17) -> D11
- U11 pad 18: unconnected-(U11-RXD0-Pad18) -> D12
- U11 pad 19: unconnected-(U11-PB7-Pad19) -> D13
- U11 pad 2: unconnected-(U11-NC-Pad2) -> A17
- U11 pad 20: unconnected-(U11-PB8-Pad20) -> D14
- U11 pad 21: unconnected-(U11-RXD1-Pad21) -> D15
- U11 pad 22: unconnected-(U11-TXD1-Pad22) -> ~{ROMH_CS}
- U11 pad 3: Net-(U11-PA0) -> A16
- U11 pad 4: Net-(U11-WP) -> A13
- U11 pad 5: Net-(U11-PA1) -> A8
- U11 pad 6: unconnected-(U11-PB6-Pad6) -> A7
- U11 pad 7: unconnected-(U11-PB9-Pad7) -> A6
- U11 pad 8: +3.3V -> A5
- U11 pad 9: unconnected-(U11-PB15-Pad9) -> A4
- U4 pad 1: unconnected-(U4-INPUT/GCLR-Pad1) -> RESET
- U4 pad 10: A23 -> (no net)
- U4 pad 11: A22 -> (no net)
- U4 pad 12: A21 -> (no net)
- U4 pad 13: +5V -> (no net)
- U4 pad 14: TDI -> +5V
- U4 pad 2: unconnected-(U4-INPUT/OE2/GCLK2-Pad2) -> ~{RESET}
- U4 pad 3: +5V -> RESET
- U4 pad 4: MPUCLOCK -> ~{HALT}
- U4 pad 5: ~{AS} -> RESET
- U4 pad 6: R/W -> Net-(R5-Pad1)
- U4 pad 8: ~{UDS} -> (no net)
- U4 pad 9: ~{LDS} -> (no net)
- U5 pad 1: A19 -> GND
- U5 pad 10: A3 -> D1
- U5 pad 11: A2 -> D2
- U5 pad 12: A1 -> D3
- U5 pad 13: D0 -> D4
- U5 pad 14: D1 -> D5
- U5 pad 15: D2 -> D6
- U5 pad 16: GND -> D7
- U5 pad 17: D3 -> unconnected-(U5-LED+-Pad17)
- U5 pad 18: D4 -> unconnected-(U5-VEE-Pad18)
- U5 pad 19: D5 -> unconnected-(U5-LED+-Pad19)
- U5 pad 2: A17 -> +5V
- U5 pad 20: D6 -> unconnected-(U5-LED--Pad20)
- U5 pad 3: A16 -> unconnected-(U5-VO-Pad3)
- U5 pad 4: A13 -> ~{VID_WR}
- U5 pad 5: A8 -> ~{VID_RD}
- U5 pad 6: A7 -> ~{VID_CS}
- U5 pad 7: A6 -> A1
- U5 pad 8: A5 -> ~{RESET}
- U5 pad 9: A4 -> D0
- U6 pad 1: D0 -> +5V
- U6 pad 10: Net-(J4-Pin_2) -> +5V
- U6 pad 11: Net-(J4-Pin_3) -> 1/2CLOCK
- U6 pad 12: +5V -> Net-(U6B-D)
- U6 pad 14: ~{UART_CS} -> +5V
- U6 pad 2: D1 -> Net-(U6A-D)
- U6 pad 3: D2 -> 1/1CLOCK
- U6 pad 4: D3 -> +5V
- U6 pad 5: D4 -> 1/2CLOCK
- U6 pad 6: D5 -> Net-(U6A-D)
- U6 pad 7: D6 -> GND
- U6 pad 8: D7 -> Net-(U6B-D)
- U6 pad 9: unconnected-(U6-RCLK-Pad9) -> 1/4CLOCK
- U7 pad 1: A19 -> Net-(U17-MP)
- U7 pad 10: A3 -> Net-(U17-CH1)
- U7 pad 11: A2 -> GND
- U7 pad 12: A1 -> Net-(U17-CH2)
- U7 pad 13: D0 -> AMP_R
- U7 pad 14: D1 -> AMP_R
- U7 pad 2: A17 -> Net-(U17-BC)
- U7 pad 3: A15 -> Net-(U17-RB)
- U7 pad 4: A13 -> +5V
- U7 pad 5: A8 -> Net-(U17-AOUT)
- U7 pad 6: A7 -> Net-(U7B--)
- U7 pad 7: A6 -> Net-(U7B--)
- U7 pad 8: A5 -> AMP_L
- U7 pad 9: A4 -> AMP_L
- U8 pad 1: GND -> +5V
- U8 pad 2: Net-(U8-TR) -> GND
- U8 pad 3: RESET -> +5V
- U8 pad 4: +5V -> GND
- U8 pad 5: GND -> +5V
- U8 pad 6: Net-(U8-DIS) -> GND
- U8 pad 7: Net-(U8-DIS) -> +5V
- U8 pad 8: +5V -> GND
- U9 pad 1: A19 -> D0
- U9 pad 10: A3 -> Net-(J4-Pin_2)
- U9 pad 11: A2 -> Net-(J4-Pin_3)
- U9 pad 12: A1 -> +5V
- U9 pad 13: D8 -> +5V
- U9 pad 14: D9 -> ~{UART_CS}
- U9 pad 15: D10 -> unconnected-(U9-~{BAUDOUT}-Pad15)
- U9 pad 16: GND -> Net-(U9-XIN)
- U9 pad 17: D11 -> unconnected-(U9-XOUT-Pad17)
- U9 pad 18: D12 -> ~{UART_WR}
- U9 pad 19: D13 -> GND
- U9 pad 2: A17 -> D1
- U9 pad 20: D14 -> GND
- U9 pad 21: D15 -> ~{UART_RD}
- U9 pad 22: ~{ROMH_CS} -> GND
- U9 pad 23: A11 -> unconnected-(U9-DDIS-Pad23)
- U9 pad 25: A12 -> unconnected-(U9-~{ADS}-Pad25)
- U9 pad 26: A10 -> A3
- U9 pad 27: A9 -> A2
- U9 pad 28: A14 -> A1
- U9 pad 29: A15 -> unconnected-(U9-~{RXRDY}-Pad29)
- U9 pad 3: A16 -> D2
- U9 pad 30: A18 -> UART_INTR
- U9 pad 32: +5V -> unconnected-(U9-~{RTS}-Pad32)
- U9 pad 4: A13 -> D3
- U9 pad 5: A8 -> D4
- U9 pad 6: A7 -> D5
- U9 pad 7: A6 -> D6
- U9 pad 8: A5 -> D7
- U9 pad 9: A4 -> unconnected-(U9-RCLK-Pad9)
- Y1 pad 1: Net-(Y1-EN) -> unconnected-(Y1-EN-Pad1)
- Y1 pad 5: Net-(U6-XIN) -> 1/1CLOCK
- Y2 pad 1: Net-(Y2-EN) -> unconnected-(Y2-EN-Pad1)
- Y2 pad 5: 1/1CLOCK -> Net-(U9-XIN)
Other:
- board outline added: 104.7 x 155.5 mm
